Commit message: WIP: improve TF tree

File: walker_description/urdf/walker_model.xacro (robot description, xacro)
@@ -1,9 +1,11 @@
 <?xml version="1.0"?>
-<robot xmlns:xacro="http://www.ros.org/wiki/xacro" name="rfid_robot">
+<robot xmlns:xacro="http://www.ros.org/wiki/xacro" name="walker">
     <!--All units in m-kg-s-radians unit system -->
-    <xacro:arg name="wheel_diameter" default="0.188"/>
-    <xacro:arg name="wheel_section" default="0.035"/>
-    <xacro:arg name="wheel_separation" default="0.5"/>
-    <xacro:arg name="lidar_height" default="0.34"/>
+    <xacro:arg name="wheel_diameter" default="0.15"/>
+    <xacro:arg name="wheel_section" default="0.022"/>
+    <xacro:arg name="wheel_separation" default="0.575"/>
+    <!-- From floor -->
+    <xacro:arg name="lidar_height" default="0.21"/>
+    <xacro:arg name="handle_height" default="0.85"/>
     <!--Constants and operable values -->
     <xacro:property name="wheel_diameter_prop" value="$(arg wheel_diameter)" />
@@ -11,10 +13,11 @@
     <xacro:property name="wheel_separation_prop" value="$(arg wheel_separation)" />
     <xacro:property name="lidar_height_prop" value="$(arg lidar_height)" />
+    <xacro:property name="handle_height_prop" value="$(arg handle_height)" />
     <xacro:property name="model_scale" value="0.0095" />
     <xacro:property name="M_PI" value="3.1415926535897931" />
     <xacro:property name="M_PI_2" value="1.570796327" />
     <!-- macros  -->
-    <xacro:macro name="link_wheel" params="name">
-        <link name="wheel_${name}_link">
+    <xacro:macro name="wheel" params="name origin_xyz">">
+        <link name="wheel_${name}">
             <inertial>
               <mass value="0.2"/>
@@ -28,5 +31,5 @@
               </geometry>
             </collision>
-            <!-- <visual name="wheel_${name}_visual">
+            <visual name="wheel_${name}_visual">
               <origin rpy="0 ${M_PI_2} ${M_PI_2}" xyz="0 0 0"/>
               <geometry>
@@ -36,47 +39,53 @@
                 <color rgba="0.0 0.0 0.0 1.0"/>
               </material>
-            </visual> -->
+            </visual>
         </link>
+        <!-- continuous type does not get done-->
+        <joint name="wheel_${name}_joint" type="fixed">
+            <origin rpy="0 0 0" xyz="${origin_xyz}"/>
+            <child link="wheel_${name}"/>
+            <parent link="base_link"/>
+            <axis rpy="0 0 0" xyz="0 1 0"/>
+            <limit effort="10000" velocity="1000"/>
+            <joint_properties damping="1.0" friction="1.0"/>
+        </joint>
     </xacro:macro>
-    <xacro:macro name="joint_wheel" params="name origin_xyz">
-      <joint name="wheel_${name}_joint" type="continuous">
-        <origin rpy="0 0 0" xyz="${origin_xyz}"/>
-        <child link="wheel_${name}_link"/>
-        <parent link="base_link"/>
-        <axis rpy="0 0 0" xyz="0 1 0"/>
-        <limit effort="10000" velocity="1000"/>
-        <joint_properties damping="1.0" friction="1.0"/>
-      </joint>
+    <xacro:macro name="handle" params="name origin_xyz">">
+        <link name="handle_${name}">
+            <inertial>
+              <mass value="0.2"/>
+              <origin rpy="0 ${M_PI_2} ${M_PI_2}" xyz="0 0 0"/>
+              <inertia ixx="0.000526666666667" ixy="0" ixz="0" iyy="0.000526666666667" iyz="0" izz="0.001"/>
+            </inertial>
+            <collision name="handle_${name}_collision">
+              <origin rpy="0 ${M_PI_2} ${M_PI_2}" xyz="0 0 0"/>
+              <geometry>
+                <cylinder radius="${wheel_diameter_prop/2}" length="${wheel_section_prop}"/>
+              </geometry>
+            </collision>
+            <visual name="handle_${name}_visual">
+              <origin rpy="0 ${M_PI_2} ${M_PI_2}" xyz="0 0 0"/>
+              <geometry>
+                <cylinder radius="${wheel_diameter_prop/2}" length="${wheel_section_prop}"/>
+              </geometry>
+              <material name="black">
+                <color rgba="0.0 0.0 0.0 1.0"/>
+              </material>
+            </visual>
+        </link>
+        <joint name="handle_${name}_joint" type="fixed">
+            <origin rpy="0 0 0" xyz="${origin_xyz}"/>
+            <child link="handle_${name}"/>
+            <parent link="base_link"/>
+            <axis rpy="0 0 0" xyz="0 1 0"/>
+            <limit effort="10000" velocity="1000"/>
+            <joint_properties damping="1.0" friction="1.0"/>
+        </joint>
     </xacro:macro>
-    <!-- gazebo stuff -->
-    <xacro:include filename="$(find walker_simulation)/urdf/walker_model.gazebo" />
+    <!-- gazebo stuff
+    <xacro:include filename="$(find walker_description)/urdf/walker_model.gazebo" />
+    -->
     <!-- root link -->
     <link name="base_footprint"/>
-    <!-- LIDAR link -->
-    <link name="base_scan">
-          <inertial>
-              <mass value="0.004" />
-              <inertia ixx="0.001" ixy="0.000" ixz="0.000" iyy="0.001" iyz="0.000" izz="0.001" />
-          </inertial>
-          <collision name="lidar_sensor_collision">
-              <geometry>
-                  <cylinder radius="0.0508" length="0.055"/>
-              </geometry>
-          </collision>
-          <visual name="lidar_sensor_visual">
-              <geometry>
-                  <mesh scale="0.001 0.001 0.001" filename="file://$(find turtlebot3_gazebo)/models/turtlebot3_burger/meshes/lds.dae"/>
-              </geometry>
-              <material name="grey">
-                <color rgba="0.2 0.2 0.2 1.0"/>
-              </material>
-          </visual>
-    </link>
-    <joint name="lidar_joint" type="fixed">
-      <origin xyz="0.0 0 ${lidar_height_prop}" rpy="0 0 0"/>
-      <axis xyz="0 0 1"/>
-      <parent link="base_link"/>
-      <child link="base_scan"/>
-    </joint>
     <!-- Chassis link -->
     <link name="base_link">
@@ -102,8 +111,35 @@
       <child link="base_link"/>
     </joint>
+    <!-- LIDAR link -->
+    <link name="laser">
+          <inertial>
+              <mass value="0.004" />
+              <inertia ixx="0.001" ixy="0.000" ixz="0.000" iyy="0.001" iyz="0.000" izz="0.001" />
+          </inertial>
+          <collision name="lidar_sensor_collision">
+              <geometry>
+                  <cylinder radius="0.0508" length="0.055"/>
+              </geometry>
+          </collision>
+          <visual name="lidar_sensor_visual">
+              <geometry>
+                  <mesh scale="0.001 0.001 0.001" filename="file://$(find turtlebot3_gazebo)/models/turtlebot3_burger/meshes/lds.dae"/>
+              </geometry>
+              <material name="grey">
+                <color rgba="0.2 0.2 0.2 1.0"/>
+              </material>
+          </visual>
+    </link>
+    <joint name="lidar_joint" type="fixed">
+      <origin xyz="0.0 0 ${lidar_height_prop}" rpy="0 0 0"/>
+      <axis xyz="0 0 1"/>
+      <parent link="base_link"/>
+      <child link="laser"/>
+    </joint>
     <!-- Wheel links -->
-    <xacro:link_wheel name="right" />
-    <xacro:joint_wheel name="right" origin_xyz="0 -${wheel_separation_prop/2} ${wheel_diameter_prop/2}" />
-    <xacro:link_wheel name="left" />
-    <xacro:joint_wheel name="left" origin_xyz="0 ${wheel_separation_prop/2} ${wheel_diameter_prop/2}" />
+    <xacro:wheel name="right" origin_xyz="0 -${wheel_separation_prop/2} ${wheel_diameter_prop/2}" />
+    <xacro:wheel name="left"  origin_xyz="0 ${wheel_separation_prop/2} ${wheel_diameter_prop/2}" />
+    <!-- Handle links -->
+    <xacro:handle name="right" origin_xyz="0.31 -0.24  ${handle_height_prop}" />
+    <xacro:handle name="left"  origin_xyz="0.31  0.24  ${handle_height_prop}" />
 </robot>

Commit message: improving tf

File: walker_description/urdf/walker_model.xacro (robot description, xacro)
@@ -2,16 +2,38 @@
 <robot xmlns:xacro="http://www.ros.org/wiki/xacro" name="walker">
     <!--All units in m-kg-s-radians unit system -->
-    <xacro:arg name="wheel_diameter" default="0.15"/>
-    <xacro:arg name="wheel_section" default="0.022"/>
-    <xacro:arg name="wheel_separation" default="0.575"/>
-    <!-- From floor -->
-    <xacro:arg name="lidar_height" default="0.21"/>
-    <xacro:arg name="handle_height" default="0.85"/>
+    <xacro:arg name="wheel_diameter_prop" default="0.15"/>
+    <xacro:arg name="wheel_section_prop" default="0.022"/>
+    <xacro:arg name="wheel_separation_prop" default="0.575"/>
+    <!-- In base_footprint coordinates:
+          0,0,0 is at floor level in the middle point between back wheels
+          x+ is towards front wheels
+          y+ is right side
+          z+ is up
+    -->
+    <xacro:arg name="lidar_pos_x_prop" default="0.55"/>
+    <xacro:arg name="lidar_pos_y_prop" default="0.0"/>
+    <xacro:arg name="lidar_pos_z_prop" default="0.21"/>
+    <xacro:arg name="witmotion_pos_x_prop" default="0.55"/>
+    <xacro:arg name="witmotion_pos_y_prop" default="0.0"/>
+    <xacro:arg name="witmotion_pos_z_prop" default="0.474"/>
+    51.3mm x36mm X15mm
+    <xacro:arg name="witmotion_size_x_prop" default="0.0513"/>
+    <xacro:arg name="witmotion_size_y_prop" default="0.036"/>
+    <xacro:arg name="witmotion_size_z_prop" default="0.015"/>
+    <!-- Handle links are managed by handle_tf_publisher.py -->
+    <!-- leapmotion link should be calculated elsewhere -->
     <!--Constants and operable values -->
-    <xacro:property name="wheel_diameter_prop" value="$(arg wheel_diameter)" />
-    <xacro:property name="wheel_section_prop" value="$(arg wheel_section)" />
-    <xacro:property name="wheel_separation_prop" value="$(arg wheel_separation)" />
-    <xacro:property name="lidar_height_prop" value="$(arg lidar_height)" />
-    <xacro:property name="handle_height_prop" value="$(arg handle_height)" />
+    <xacro:property name="wheel_diameter" value="$(arg wheel_diameter_prop)" />
+    <xacro:property name="wheel_section" value="$(arg wheel_section_prop)" />
+    <xacro:property name="wheel_separation" value="$(arg wheel_separation_prop)" />
+    <xacro:property name="lidar_pos_x" value="$(arg lidar_pos_x_prop)" />
+    <xacro:property name="lidar_pos_y" value="$(arg lidar_pos_y_prop)" />
+    <xacro:property name="lidar_pos_z" value="$(arg lidar_pos_z_prop)" />
+    <xacro:property name="witmotion_pos_x" value="$(arg witmotion_pos_x_prop)" />
+    <xacro:property name="witmotion_pos_y" value="$(arg witmotion_pos_y_prop)" />
+    <xacro:property name="witmotion_pos_z" value="$(arg witmotion_pos_z_prop)" />
+    <xacro:property name="witmotion_size_x" value="$(arg witmotion_size_x_prop)" />
+    <xacro:property name="witmotion_size_y" value="$(arg witmotion_size_y_prop)" />
+    <xacro:property name="witmotion_size_z" value="$(arg witmotion_size_z_prop)" />
     <xacro:property name="model_scale" value="0.0095" />
     <xacro:property name="M_PI" value="3.1415926535897931" />
@@ -28,5 +50,5 @@
               <origin rpy="0 ${M_PI_2} ${M_PI_2}" xyz="0 0 0"/>
               <geometry>
-                <cylinder radius="${wheel_diameter_prop/2}" length="${wheel_section_prop}"/>
+                <cylinder radius="${wheel_diameter/2}" length="${wheel_section}"/>
               </geometry>
             </collision>
@@ -34,5 +56,5 @@
               <origin rpy="0 ${M_PI_2} ${M_PI_2}" xyz="0 0 0"/>
               <geometry>
-                <cylinder radius="${wheel_diameter_prop/2}" length="${wheel_section_prop}"/>
+                <cylinder radius="${wheel_diameter/2}" length="${wheel_section}"/>
               </geometry>
               <material name="black">
@@ -51,39 +73,4 @@
         </joint>
     </xacro:macro>
-    <xacro:macro name="handle" params="name origin_xyz">">
-        <link name="handle_${name}">
-            <inertial>
-              <mass value="0.2"/>
-              <origin rpy="0 ${M_PI_2} ${M_PI_2}" xyz="0 0 0"/>
-              <inertia ixx="0.000526666666667" ixy="0" ixz="0" iyy="0.000526666666667" iyz="0" izz="0.001"/>
-            </inertial>
-            <collision name="handle_${name}_collision">
-              <origin rpy="0 ${M_PI_2} ${M_PI_2}" xyz="0 0 0"/>
-              <geometry>
-                <cylinder radius="${wheel_diameter_prop/2}" length="${wheel_section_prop}"/>
-              </geometry>
-            </collision>
-            <visual name="handle_${name}_visual">
-              <origin rpy="0 ${M_PI_2} ${M_PI_2}" xyz="0 0 0"/>
-              <geometry>
-                <cylinder radius="${wheel_diameter_prop/2}" length="${wheel_section_prop}"/>
-              </geometry>
-              <material name="black">
-                <color rgba="0.0 0.0 0.0 1.0"/>
-              </material>
-            </visual>
-        </link>
-        <joint name="handle_${name}_joint" type="fixed">
-            <origin rpy="0 0 0" xyz="${origin_xyz}"/>
-            <child link="handle_${name}"/>
-            <parent link="base_link"/>
-            <axis rpy="0 0 0" xyz="0 1 0"/>
-            <limit effort="10000" velocity="1000"/>
-            <joint_properties damping="1.0" friction="1.0"/>
-        </joint>
-    </xacro:macro>
-    <!-- gazebo stuff
-    <xacro:include filename="$(find walker_description)/urdf/walker_model.gazebo" />
-    -->
     <!-- root link -->
     <link name="base_footprint"/>
@@ -97,18 +84,21 @@
           <collision name="base_collision">
               <geometry>
-                  <mesh scale="${model_scale} ${model_scale} ${5*model_scale/6}" filename="file://$(find walker_simulation)/models/walker/walker_no_wheels.dae"/>
+                  <mesh scale="${model_scale} ${model_scale} ${5*model_scale/6}" filename="file://$(find walker_description)/models/walker/walker_no_wheels.dae"/>
               </geometry>
           </collision>
           <visual name="base_visual">
               <geometry>
-                  <mesh scale="${model_scale} ${model_scale} ${5*model_scale/6}" filename="file://$(find walker_simulation)/models/walker/walker.dae"/>
+                  <mesh scale="${model_scale} ${model_scale} ${5*model_scale/6}" filename="file://$(find walker_description)/models/walker/walker.dae"/>
               </geometry>
           </visual>
     </link>
     <joint name="base_joint" type="fixed">
-      <origin xyz="0 0 0.01" rpy="0 0 0"/>
+      <origin xyz="0 0 ${wheel_diameter/2}" rpy="0 0 0"/>
       <parent link="base_footprint"/>
       <child link="base_link"/>
     </joint>
+    <!-- Wheel links -->
+    <xacro:wheel name="right" origin_xyz="0 -${wheel_separation/2} ${wheel_diameter/2}" />
+    <xacro:wheel name="left"  origin_xyz="0 ${wheel_separation/2} ${wheel_diameter/2}" />
     <!-- LIDAR link -->
     <link name="laser">
@@ -124,5 +114,5 @@
           <visual name="lidar_sensor_visual">
               <geometry>
-                  <mesh scale="0.001 0.001 0.001" filename="file://$(find turtlebot3_gazebo)/models/turtlebot3_burger/meshes/lds.dae"/>
+                  <mesh scale="0.001 0.001 0.001" filename="file://$(find walker_description)/models/turtlebot3_burger/meshes/lds.dae"/>
               </geometry>
               <material name="grey">
@@ -132,14 +122,37 @@
     </link>
     <joint name="lidar_joint" type="fixed">
-      <origin xyz="0.0 0 ${lidar_height_prop}" rpy="0 0 0"/>
+      <origin xyz="${lidar_pos_x} ${lidar_pos_y} ${lidar_pos_z}" rpy="0 0 0"/>
       <axis xyz="0 0 1"/>
-      <parent link="base_link"/>
+      <parent link="base_footprint"/>
       <child link="laser"/>
     </joint>
-    <!-- Wheel links -->
-    <xacro:wheel name="right" origin_xyz="0 -${wheel_separation_prop/2} ${wheel_diameter_prop/2}" />
-    <xacro:wheel name="left"  origin_xyz="0 ${wheel_separation_prop/2} ${wheel_diameter_prop/2}" />
-    <!-- Handle links -->
-    <xacro:handle name="right" origin_xyz="0.31 -0.24  ${handle_height_prop}" />
-    <xacro:handle name="left"  origin_xyz="0.31  0.24  ${handle_height_prop}" />
+    <!-- IMU link -->
+    <link name="witmotion">
+          <inertial>
+              <mass value="0.004" />
+              <inertia ixx="0.001" ixy="0.000" ixz="0.000" iyy="0.001" iyz="0.000" izz="0.001" />
+          </inertial>
+          <collision name="witmotion_sensor_collision">
+              <geometry>
+                  <box size="${witmotion_size_x} ${witmotion_size_y} ${witmotion_size_z}"/>
+              </geometry>
+          </collision>
+          <visual name="witmotion_sensor_visual">
+              <geometry>
+                  <box size="${witmotion_size_x} ${witmotion_size_y} ${witmotion_size_z}"/>
+              </geometry>
+              <material name="grey">
+                <color rgba="0.2 0.2 0.2 1.0"/>
+              </material>
+          </visual>
+    </link>
+    <joint name="witmotion_joint" type="fixed">
+      <origin xyz="${witmotion_pos_x+witmotion_size_x/2} ${witmotion_pos_y+witmotion_size_y/2} ${witmotion_pos_z+witmotion_size_z/2}" rpy="0 0 0"/>
+      <axis xyz="0 0 1"/>
+      <parent link="base_footprint"/>
+      <child link="witmotion"/>
+    </joint>
+    <!-- gazebo stuff
+    <xacro:include filename="$(find walker_description)/urdf/walker_model.gazebo" />
+    -->
 </robot>

Commit message: mch2

File: walker_description/urdf/walker_model.xacro (robot description, xacro)
@@ -17,5 +17,4 @@
     <xacro:arg name="witmotion_pos_y_prop" default="0.0"/>
     <xacro:arg name="witmotion_pos_z_prop" default="0.474"/>
-    51.3mm x36mm X15mm
     <xacro:arg name="witmotion_size_x_prop" default="0.0513"/>
     <xacro:arg name="witmotion_size_y_prop" default="0.036"/>
@@ -36,5 +35,7 @@
     <xacro:property name="witmotion_size_y" value="$(arg witmotion_size_y_prop)" />
     <xacro:property name="witmotion_size_z" value="$(arg witmotion_size_z_prop)" />
-    <xacro:property name="model_scale" value="0.0095" />
+    <xacro:property name="model_scale_x" value="0.01" />
+    <xacro:property name="model_scale_y" value="0.0095" />
+    <xacro:property name="model_scale_z" value="0.0095" />
     <xacro:property name="M_PI" value="3.1415926535897931" />
     <xacro:property name="M_PI_2" value="1.570796327" />
@@ -67,5 +68,5 @@
             <origin rpy="0 0 0" xyz="${origin_xyz}"/>
             <child link="wheel_${name}"/>
-            <parent link="base_link"/>
+            <parent link="base_footprint"/>
             <axis rpy="0 0 0" xyz="0 1 0"/>
             <limit effort="10000" velocity="1000"/>
@@ -84,10 +85,10 @@
           <collision name="base_collision">
               <geometry>
-                  <mesh scale="${model_scale} ${model_scale} ${5*model_scale/6}" filename="file://$(find walker_description)/models/walker/walker_no_wheels.dae"/>
+                  <mesh scale="${model_scale_x} ${model_scale_y} ${model_scale_z}" filename="package://walker_description/models/walker/walker_no_wheels.dae"/>
               </geometry>
           </collision>
           <visual name="base_visual">
               <geometry>
-                  <mesh scale="${model_scale} ${model_scale} ${5*model_scale/6}" filename="file://$(find walker_description)/models/walker/walker.dae"/>
+                  <mesh scale="${model_scale_x} ${model_scale_y} ${model_scale_z}" filename="package://walker_description/models/walker/walker.dae"/>
               </geometry>
           </visual>
@@ -114,5 +115,5 @@
           <visual name="lidar_sensor_visual">
               <geometry>
-                  <mesh scale="0.001 0.001 0.001" filename="file://$(find walker_description)/models/turtlebot3_burger/meshes/lds.dae"/>
+                  <mesh scale="0.001 0.001 0.001" filename="package://walker_description/models/turtlebot3_burger/meshes/lds.dae"/>
               </geometry>
               <material name="grey">
@@ -154,5 +155,5 @@
     </joint>
     <!-- gazebo stuff
-    <xacro:include filename="$(find walker_description)/urdf/walker_model.gazebo" />
+    <xacro:include filename="package://walker_description/urdf/walker_model.gazebo" />
     -->
 </robot>

Commit message: New robot model. New tf tree. New gui. Needs some testing

File: walker_description/urdf/walker_model.xacro (robot description, xacro)
@@ -5,4 +5,5 @@
     <xacro:arg name="wheel_section_prop" default="0.022"/>
     <xacro:arg name="wheel_separation_prop" default="0.575"/>
+    <xacro:arg name="back_front_wheel_separation_prop" default="0.53"/>
     <!-- In base_footprint coordinates:
           0,0,0 is at floor level in the middle point between back wheels
@@ -26,4 +27,5 @@
     <xacro:property name="wheel_section" value="$(arg wheel_section_prop)" />
     <xacro:property name="wheel_separation" value="$(arg wheel_separation_prop)" />
+    <xacro:property name="back_front_wheel_separation" value="$(arg back_front_wheel_separation_prop)" />
     <xacro:property name="lidar_pos_x" value="$(arg lidar_pos_x_prop)" />
     <xacro:property name="lidar_pos_y" value="$(arg lidar_pos_y_prop)" />
@@ -35,7 +37,7 @@
     <xacro:property name="witmotion_size_y" value="$(arg witmotion_size_y_prop)" />
     <xacro:property name="witmotion_size_z" value="$(arg witmotion_size_z_prop)" />
-    <xacro:property name="model_scale_x" value="0.01" />
-    <xacro:property name="model_scale_y" value="0.0095" />
-    <xacro:property name="model_scale_z" value="0.0095" />
+    <xacro:property name="model_scale_x" value="0.009" /> <!--long -->
+    <xacro:property name="model_scale_y" value="0.0105" /> <!--wide -->
+    <xacro:property name="model_scale_z" value="0.0075" /> <!--high -->
     <xacro:property name="M_PI" value="3.1415926535897931" />
     <xacro:property name="M_PI_2" value="1.570796327" />
@@ -84,4 +86,5 @@
           </inertial>
           <collision name="base_collision">
+              <origin rpy="0 0 0" xyz="${back_front_wheel_separation} 0.0 -${wheel_diameter/2}"/>
               <geometry>
                   <mesh scale="${model_scale_x} ${model_scale_y} ${model_scale_z}" filename="package://walker_description/models/walker/walker_no_wheels.dae"/>
@@ -89,4 +92,5 @@
           </collision>
           <visual name="base_visual">
+              <origin rpy="0 0 0" xyz="${back_front_wheel_separation} 0.0 -${wheel_diameter/2}"/>
               <geometry>
                   <mesh scale="${model_scale_x} ${model_scale_y} ${model_scale_z}" filename="package://walker_description/models/walker/walker.dae"/>
