Commit message: WIP: adding d435 and new imu sw to system

File: walker_description/urdf/walker_model.xacro (robot description, xacro)
@@ -21,4 +21,7 @@
     <xacro:arg name="witmotion_size_y_prop" default="0.036"/>
     <xacro:arg name="witmotion_size_z_prop" default="0.015"/>
+    <xacro:arg name="camera_pos_x_prop" default="0.6"/>
+    <xacro:arg name="camera_pos_y_prop" default="0.00"/>
+    <xacro:arg name="camera_pos_z_prop" default="0.305"/>
     <!-- Handle links are managed by handle_tf_publisher.py -->
     <!-- leapmotion link should be calculated elsewhere -->
@@ -37,4 +40,7 @@
     <xacro:property name="witmotion_size_y" value="$(arg witmotion_size_y_prop)" />
     <xacro:property name="witmotion_size_z" value="$(arg witmotion_size_z_prop)" />
+    <xacro:property name="camera_pos_x" value="$(arg camera_pos_x_prop)" />
+    <xacro:property name="camera_pos_y" value="$(arg camera_pos_y_prop)" />
+    <xacro:property name="camera_pos_z" value="$(arg camera_pos_z_prop)" />
     <xacro:property name="model_scale_x" value="0.009" /> <!--long -->
     <xacro:property name="model_scale_y" value="0.0105" /> <!--wide -->
@@ -43,5 +49,5 @@
     <xacro:property name="M_PI_2" value="1.570796327" />
     <!-- macros  -->
-    <xacro:macro name="wheel" params="name origin_xyz">">
+    <xacro:macro name="wheel" params="name origin_xyz">
         <link name="wheel_${name}">
             <inertial>
@@ -153,9 +159,14 @@
     </link>
     <joint name="witmotion_joint" type="fixed">
-      <origin xyz="${witmotion_pos_x+witmotion_size_x/2} ${witmotion_pos_y+witmotion_size_y/2} ${witmotion_pos_z+witmotion_size_z/2}" rpy="0 0 0"/>
+      <origin xyz="${witmotion_pos_x} ${witmotion_pos_y} ${witmotion_pos_z}" rpy="0 0 0"/>
       <axis xyz="0 0 1"/>
       <parent link="base_footprint"/>
       <child link="witmotion"/>
     </joint>
+     <!-- realsense camera -->
+    <xacro:include filename="$(find realsense2_description)/urdf/_d435.urdf.xacro"/>
+    <xacro:sensor_d435 name="camera" parent="base_footprint">
+      <origin xyz="${camera_pos_x} ${camera_pos_y} ${camera_pos_z}" rpy="0 0 0"/>
+    </xacro:sensor_d435>
     <!-- gazebo stuff
     <xacro:include filename="package://walker_description/urdf/walker_model.gazebo" />

Commit message: - changed to ros2 branch of the official rplidar repo - moved tmule config files to its own folder - changed imu node to achieve 100Hz - WIP: ekf odometry fusion

File: walker_description/urdf/walker_model.xacro (robot description, xacro)
@@ -18,4 +18,7 @@
     <xacro:arg name="witmotion_pos_y_prop" default="0.0"/>
     <xacro:arg name="witmotion_pos_z_prop" default="0.305"/>
+    <xacro:arg name="witmotion_pos_roll_prop" default="180.0"/>
+    <xacro:arg name="witmotion_pos_pitch_prop" default="0.0"/>
+    <xacro:arg name="witmotion_pos_yaw_prop" default="0.0"/>
     <xacro:arg name="witmotion_size_x_prop" default="0.0513"/>
     <xacro:arg name="witmotion_size_y_prop" default="0.036"/>
@@ -37,4 +40,7 @@
     <xacro:property name="witmotion_pos_y" value="$(arg witmotion_pos_y_prop)" />
     <xacro:property name="witmotion_pos_z" value="$(arg witmotion_pos_z_prop)" />
+    <xacro:property name="witmotion_pos_roll" value="$(arg witmotion_pos_roll_prop)" />
+    <xacro:property name="witmotion_pos_pitch" value="$(arg witmotion_pos_pitch_prop)" />
+    <xacro:property name="witmotion_pos_yaw" value="$(arg witmotion_pos_yaw_prop)" />
     <xacro:property name="witmotion_size_x" value="$(arg witmotion_size_x_prop)" />
     <xacro:property name="witmotion_size_y" value="$(arg witmotion_size_y_prop)" />
@@ -159,5 +165,5 @@
     </link>
     <joint name="witmotion_joint" type="fixed">
-      <origin xyz="${witmotion_pos_x} ${witmotion_pos_y} ${witmotion_pos_z}" rpy="0 0 0"/>
+      <origin xyz="${witmotion_pos_x} ${witmotion_pos_y} ${witmotion_pos_z}" rpy="${witmotion_pos_roll*M_PI_2/90} ${witmotion_pos_pitch*M_PI_2/90} ${witmotion_pos_yaw*M_PI_2/90}"/>
       <axis xyz="0 0 1"/>
       <parent link="base_footprint"/>
